Commit message: fixed lidar and differntial

File: urdf/AMR_1.xacro (robot description, xacro)
@@ -68,5 +68,5 @@
     </collision>
   </link>
-  <link name="lidar_link">
+  <!-- <link name="lidar_link">
     <inertial>
       <origin xyz="0.0084954458305041 -0.09792752116058154 0.4033086335221119" rpy="0 0 0" />
@@ -89,4 +89,20 @@
       </geometry>
     </collision>
+  </link> -->
+  <link name="lidar_link">
+    <visual>
+      <geometry>
+        <cylinder radius="0.05" length="0.04" />
+      </geometry>
+    </visual>
+    <collision>
+      <geometry>
+        <cylinder radius="0.05" length="0.04" />
+      </geometry>
+    </collision>
+    <inertial>
+      <mass value="0.5" />
+      <inertia ixx="0.000252666666667" ixy="0" ixz="0" iyy="0.000252666666667" iyz="0" izz="0.0005" />
+    </inertial>
   </link>
   <joint name="Revolute_3" type="continuous">
@@ -103,5 +119,5 @@
   </joint>
   <joint name="Rigid_5" type="fixed">
-    <origin xyz="0.205 0.1 -0.125" rpy="0 0 0" />
+    <origin xyz="0.25 0 0.27" rpy="0 0 0" />
     <parent link="base_link" />
     <child link="lidar_link" />

Commit message: gmapping module done and also transforms are corrected

File: urdf/AMR_1.xacro (robot description, xacro)
@@ -106,4 +106,6 @@
     </inertial>
   </link>
+  <link name="robot_footprint">
+  </link>
   <joint name="Revolute_3" type="continuous">
     <origin xyz="-0.097072 -0.202928 0.049293" rpy="0 0 0" />
@@ -123,3 +125,7 @@
     <child link="lidar_link" />
   </joint>
+  <joint name="dummy_joint" type="fixed">
+    <parent link="robot_footprint" />
+    <child link="base_link" />
+  </joint>
 </robot>
